File: schematics/Display device/Display device.kicad_pcb (KiCad board)
At the start: 2 copper layers, 57.5 x 44.5 mm, 11 parts, among them J1 stepper motor, SW1 SW_Push, U1 XIAO ESP32C3

Commit message: kicad update
Parts:
- moved U1 46.0 mm to (100.9, 56.4)
- moved C1 46.0 mm to (101.0, 80.0)
- moved C2 46.0 mm to (101.0, 83.5)
- moved D1 46.0 mm to (81.5, 49.5)
- moved J1 46.0 mm to (128.5, 64.3)
- moved R1 46.0 mm to (84.5, 49.5)
- moved R2 46.0 mm to (119.0, 64.0)
- moved R3 46.0 mm to (119.0, 61.5)
- moved R4 46.0 mm to (119.0, 59.0)
- moved R5 46.0 mm to (119.0, 56.5)
- moved SW1 46.0 mm to (83.2, 75.5)

Commit message: sche update
Parts:
- removed J1: stepper motor, Connector_PinHeader_2.54mm:PinHeader_1x04_P2.54mm_Vertical
- added M1: Stepper_Motor_bipolar, x27_Footprint:x27_stepper_two_holes, F.Cu at (116.5, 54.0)
- added REF1: MountingHole_2.5mm, MountingHole:MountingHole_2.5mm, F.Cu at (59.0, 79.5)
- added REF2: MountingHole_2.5mm, MountingHole:MountingHole_2.5mm, F.Cu at (133.5, 48.5)
- SW1: footprint Button_Switch_SMD:SW_Push_1P1T_NO_E-Switch_TL3301NxxxxxG -> Button_Switch_SMD:SW_SPST_EVQP7A
- moved SW1 31.1 mm to (54.2, 64.3)
- moved C1 23.6 mm to (77.4, 79.2)
- moved C2 23.6 mm to (77.4, 82.7)
- moved R2 23.6 mm to (95.4, 63.1)
- moved R3 23.6 mm to (95.4, 60.6)
- moved R4 23.6 mm to (95.4, 58.1)
- moved R5 23.6 mm to (95.4, 55.6)
- moved U1 23.6 mm to (77.3, 55.5)
- moved D1 23.6 mm to (57.9, 48.6)
- moved R1 23.6 mm to (60.9, 48.6)
Routing:
- net Net-(M1-Pad3): track 8.60 -> 38.1 mm
- net Net-(M1-Pad4): track 8.58 -> 36.5 mm
- net /DISP_BTN: track 27.4 -> 21.2 mm
- net Net-(M1-Pad1): track 8.63 -> 13.2 mm
- net Net-(M1--): track 8.61 -> 11.3 mm
Other:
- board size 57.5 x 44.5 mm -> 87 x 43 mm
- board text added: "Polly Yao EmoTrace 2.0"
- board text removed: "Polly Yao EmoTrace 1.0"
